File: cyclops.kicad_pcb (KiCad board)
At the start: 2 copper layers, 136 parts, among them J1 USB_mini_micro_B, K1 ESC, K10 KEYSW, K11 KEYSW, K12 KEYSW, K13 KEYSW, K14 backspace, K15 tab, K16 KEYSW, K17 KEYSW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

Commit message: Clean some routing
Routing:
- net /COL5: track 84.1 -> 87.7 mm
- net /COL2: track 145.0 -> 142.8 mm
- net /COL3: track 108.3 -> 109.5 mm
- net /ROW3: track 263.2 -> 262.3 mm
